File: mcuDevBoard.kicad_pcb (KiCad board)
At the start: 2 copper layers, 112 x 51 mm, 110 parts, among them J1 Conn_01x02, J12 display1, J13 display2, J15 Conn_01x03, J2 Conn_01x16, J3 USB_C_Receptacle_USB2.0, J4 Conn_01x16, J5 Conn_01x16, J6 power input, J7 Conn_01x16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

Commit message: pcb v0.2
Parts:
- removed R39, R40: 0, Resistor_SMD:R_0805_2012Metric
- added J10: motorDriver, Connector_PinHeader_2.54mm:PinHeader_1x04_P2.54mm_Vertical, F.Cu at (117.6, 98.5)
- added JP13: JO, Jumper:SolderJumper-2_P1.3mm_Open_RoundedPad1.0x1.5mm, B.Cu at (87.2, 95.0)
- added JP14: JO, Jumper:SolderJumper-2_P1.3mm_Open_RoundedPad1.0x1.5mm, B.Cu at (155.2, 97.3)
- added JP15: JO, Jumper:SolderJumper-2_P1.3mm_Open_RoundedPad1.0x1.5mm, F.Cu at (116.8, 104.5)
- added JP17: SolderJumper_2_Bridged, Jumper:SolderJumper-2_P1.3mm_Bridged_RoundedPad1.0x1.5mm, B.Cu at (87.3, 99.0)
- added JP18: SolderJumper_2_Bridged, Jumper:SolderJumper-2_P1.3mm_Bridged_RoundedPad1.0x1.5mm, B.Cu at (155.2, 100.1)
- added JP19: ledVoltage, Jumper:SolderJumper-2_P1.3mm_Bridged_RoundedPad1.0x1.5mm, F.Cu at (112.8, 104.5)
- C12, C13: footprint Capacitor_SMD:C_0402_1005Metric_Pad0.74x0.62mm_HandSolder -> Capacitor_SMD:C_0805_2012Metric_Pad1.18x1.45mm_HandSolder
- J6: footprint Easyeda2kicad:CONN-TH_4P-P7.50_DIBO_DB128V-7.5-4P-GN-S -> easyeda2kicad:CONN-TH_4P-P7.50_DIBO_DB128V-7.5-4P-GN-S
- moved R41 9.54 mm to (115.0, 109.5)
- moved R42 9.51 mm to (117.5, 109.5)
- moved Q1 6.86 mm to (121.6, 109.0), turned to 0 degrees
- moved J15 3.62 mm to (120.1, 114.3)
- moved J6 2.01 mm to (98.2, 74.5)
- moved J13 0.85 mm to (143.6, 99.6)
- moved C12 0.82 mm to (126.5, 84.1)
- moved C13 0.70 mm to (130.5, 94.5)
- moved R72 0.43 mm to (103.7, 105.8)
- moved J7 0.33 mm to (68.1, 110.5)
- moved J8 0.33 mm to (68.1, 115.6)
- moved J9 0.33 mm to (68.1, 113.0)
- moved J2 0.28 mm to (136.1, 110.5)
- moved J4 0.28 mm to (136.1, 115.6)
- moved J5 0.28 mm to (136.1, 113.0)
Connections:
- U1 pad 30: unconnected-(U1-GPIO19-Pad30) -> RX
- U1 pad 31: unconnected-(U1-GPIO20-Pad31) -> TX
- U1 pad 37: unconnected-(U1-GPIO25-Pad37) -> M_CLK1
- U1 pad 6: unconnected-(U1-GPIO4-Pad6) -> M_CLK2
- U2 pad 25: GND -> Net-(JP14-A)
- U6 pad 25: GND -> Net-(JP13-A)
Routing:
- net GND: track 402.2 -> 230.6 mm
- net M_CLK2: track 0.00 -> 44.0 mm
- net M_CLK1: track 0.00 -> 37.6 mm, vias 0 -> 2
- net +12V: track 99.7 -> 124.4 mm, vias 1 -> 0
- net +3.3V: track 210.7 -> 230.6 mm, vias 10 -> 11
- net TX: track 0.00 -> 11.5 mm
- net ledHigh: track 23.0 -> 13.3 mm
- net RX: track 0.00 -> 8.74 mm
- net +5V: track 119.7 -> 111.1 mm, vias 3 -> 2
- net Net-(JP13-A): track 0.00 -> 7.89 mm, vias 0 -> 1
- net VBUS: track 7.64 -> 14.9 mm
- net Net-(JP14-A): track 0.00 -> 6.79 mm, vias 0 -> 1
- net ledVcc: track 19.6 -> 13.1 mm
- net GPIO12: track 37.4 -> 38.9 mm
- net ledLow: track 20.9 -> 22.2 mm
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