File: mcuDevBoard.kicad_sch (KiCad schematic)
At the start: 40 parts, among them J1 Conn_01x02, J12 display1, J13 display2, J15 Conn_01x03, J3 USB_C_Receptacle_USB2.0, J6 power input, Q1 NMOS, U1 RP2040, U3 NCP1117-3.3_SOT223, U4 USBLC6-2SC6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

Commit message: pcb v0.2
Parts:
- removed R39, R40: 0, Resistor_SMD:R_0805_2012Metric, symbol Device:R
- added J10: motorDriver, Connector_PinHeader_2.54mm:PinHeader_1x04_P2.54mm_Vertical, symbol Connector:Conn_01x04_Pin
- added JP15: JO, Jumper:SolderJumper-2_P1.3mm_Open_RoundedPad1.0x1.5mm, symbol Jumper:SolderJumper_2_Open
- added JP19: ledVoltage, Jumper:SolderJumper-2_P1.3mm_Bridged_RoundedPad1.0x1.5mm, symbol Jumper:SolderJumper_2_Bridged
- C12, C13: footprint Capacitor_SMD:C_0402_1005Metric_Pad0.74x0.62mm_HandSolder -> Capacitor_SMD:C_0805_2012Metric_Pad1.18x1.45mm_HandSolder
- J6: footprint Easyeda2kicad:CONN-TH_4P-P7.50_DIBO_DB128V-7.5-4P-GN-S -> easyeda2kicad:CONN-TH_4P-P7.50_DIBO_DB128V-7.5-4P-GN-S
Connections:
- net +12V: now also JP15.1 (A)
- net +3.3V: now also J10.4 (Pin_4)
- net +5V: now also JP19.1 (A)
- net GND: now also J10.1 (Pin_1)
- net ledVcc: now also JP15.2 (B), JP19.2 (B)
- net RX: now reaches U1.30 (GPIO19)
- net RX: now also J10.2 (Pin_2)
- net TX: now reaches U1.31 (GPIO20)
- net TX: now also J10.3 (Pin_3)
- net M_CLK1: now reaches U1.37 (GPIO25)
- net M_CLK2: now reaches U1.6 (GPIO4)
- no-connect marks 27 -> 22
Other:
- sheet servoMultiplexer ports: added EXT_CLK; removed none
- sheet servoMultiplexer1 ports: added EXT_CLK; removed none
- moved on the sheet: J12, J13
