File: servoMultiplexer.kicad_sch (KiCad schematic)
At the start: 35 parts, among them J7 Conn_01x16, J8 Conn_01x16, J9 Conn_01x16, U6 PCA9685PW

Commit message: pcb v0.2
Parts:
- added JP13: JO, Jumper:SolderJumper-2_P1.3mm_Open_RoundedPad1.0x1.5mm, symbol Jumper:SolderJumper_2_Open
- added JP17: SolderJumper_2_Bridged, Jumper:SolderJumper-2_P1.3mm_Bridged_RoundedPad1.0x1.5mm, symbol Jumper:SolderJumper_2_Bridged
Connections:
- net GND: now also JP17.2 (B); no longer U6.25 (EXTCLK)
- new net: JP13.1 (A), JP17.1 (A), U6.25 (EXTCLK)
- new net EXT_CLK: JP13.2 (B)
Changed lines of the file:
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@@
 (kicad_sch
-	(version 20231120)
+	(version 20250114)
 	(generator "eeschema")
-	(generator_version "8.0")
+	(generator_version "9.0")
 	(paper "A4")
 	(junction
@@
 	)
 	(junction
+		(at 43.18 57.15)
+		(diameter 0)
+		(color 0 0 0 0)
+	)
+	(junction
 		(at 161.29 87.63)
 		(diameter 0)
@@
 	(wire
 		(pts
+			(xy 31.75 57.15) (xy 35.56 57.15)
+		)
+		(stroke
+			(width 0)
+			(type default)
+		)
+	)
+	(wire
+		(pts
 			(xy 50.8 77.47) (xy 50.8 80.01)
 		)
@@
 	(wire
 		(pts
-			(xy 48.26 57.15) (xy 50.8 57.15)
+			(xy 43.18 57.15) (xy 50.8 57.15)
 		)
 		(stroke
@@
 		)
 	)
+	(hierarchical_label "EXT_CLK"
+		(shape input)
+		(at 31.75 57.15 180)
+		(effects
+			(font
+				(size 1.27 1.27)
+			)
+			(justify right)
+		)
+	)
 	(hierarchical_label "SCL"
 		(shape input)
 		(at 60.96 52.07 180)
-		(fields_autoplaced yes)
 		(effects
 			(font
@@
 		(shape input)
 		(at 182.88 92.71 270)
-		(fields_autoplaced yes)
 		(effects
 			(font
@@
 		(shape input)
 		(at 60.96 54.61 180)
-		(fields_autoplaced yes)
 		(effects
 			(font
@@
 	(symbol
 		(lib_id "power:GND")
-		(at 48.26 57.15 270)
+		(at 43.18 49.53 180)
 		(unit 1)
 		(exclude_from_sim no)
@@
 		(fields_autoplaced yes)
 		(property "Reference" "#PWR042"
-			(at 41.91 57.15 0)
+			(at 43.18 43.18 0)
 			(effects
 				(font
@@
 		)
 		(property "Value" "GND"
-			(at 44.45 57.1499 90)
+			(at 45.72 48.2599 0)
 			(effects
 				(font
@@
 		)
 		(property "Footprint" ""
-			(at 48.26 57.15 0)
+			(at 43.18 49.53 0)
 			(effects
 				(font
@@
 		)
 		(property "Datasheet" ""
-			(at 48.26 57.15 0)
+			(at 43.18 49.53 0)
 			(effects
 				(font
@@
 		)
 		(property "Description" "Power symbol creates a global label with name \"GND\" , ground"
-			(at 48.26 57.15 0)
+			(at 43.18 49.53 0)
 			(effects
 				(font
@@
 	)
 	(symbol
+		(lib_id "Jumper:SolderJumper_2_Bridged")
+		(at 43.18 53.34 90)
+		(unit 1)
+		(exclude_from_sim yes)
+		(in_bom no)
+		(on_board yes)
+		(dnp no)
+		(property "Reference" "JP17"
+			(at 45.72 52.0699 90)
+			(effects
+				(font
+					(size 1.27 1.27)
+				)
+				(justify right)
+			)
+		)
+		(property "Value" "SolderJumper_2_Bridged"
+			(at 27.178 41.656 90)
+			(effects
+				(font
+					(size 1.27 1.27)
+				)
+				(justify right)
+			)
+		)
+		(property "Footprint" "Jumper:SolderJumper-2_P1.3mm_Bridged_RoundedPad1.0x1.5mm"
+			(at 43.18 53.34 0)
+			(effects
+				(font
+					(size 1.27 1.27)
+				)
+				(hide yes)
+			)
+		)
+		(property "Datasheet" "~"
+			(at 43.18 53.34 0)
+			(effects
+				(font
+					(size 1.27 1.27)
+				)
+				(hide yes)
+			)
+		)
+		(property "Description" "Solder Jumper, 2-pole, closed/bridged"
+			(at 43.18 53.34 0)
+			(effects
+				(font
+					(size 1.27 1.27)
+				)
+				(hide yes)
+			)
+		)
+		(pin "1"
+		)
+		(pin "2"
+		)
+		(instances
+			(project ""
+				(path "/76df3d58-0caf-44f2-90e9-e1295852820b/5d32edae-5069-49d0-8f93-a70e744e16c2"
+					(reference "JP17")
+					(unit 1)
+				)
+				(path "/76df3d58-0caf-44f2-90e9-e1295852820b/701c2a91-874a-4ca7-8c4e-53a7a8712d0a"
+					(reference "JP18")
+					(unit 1)
+				)
+			)
+		)
+	)
+	(symbol
 		(lib_id "Connector_Generic:Conn_01x16")
 		(at 187.96 69.85 0)
@@
 		)
 		(property "Value" "PWR_FLAG"
-			(at 45.974 52.578 0)
+			(at 53.848 46.482 0)
 			(effects
 				(font
@@
 					(unit 1)
 				)
+			)
+		)
+	)
+	(symbol
+		(lib_id "Jumper:SolderJumper_2_Open")
+		(at 39.37 57.15 180)
+		(unit 1)
+		(exclude_from_sim yes)
+		(in_bom no)
+		(on_board yes)
+		(dnp no)
+		(property "Reference" "JP13"
+			(at 35.052 63.246 0)
+			(effects
+				(font
+					(size 1.27 1.27)
+				)
+			)
+		)
+		(property "Value" "JO"
+			(at 35.052 60.706 0)
+			(effects
+				(font
+					(size 1.27 1.27)
+				)
+			)
+		)
+		(property "Footprint" "Jumper:SolderJumper-2_P1.3mm_Open_RoundedPad1.0x1.5mm"
+			(at 39.37 57.15 0)
+			(effects
+				(font
+					(size 1.27 1.27)
+				)
+				(hide yes)
+			)
+		)
+		(property "Datasheet" "~"
+			(at 39.37 57.15 0)
+			(effects
+				(font
+					(size 1.27 1.27)
+				)
+				(hide yes)
+			)
+		)
+		(property "Description" "Solder Jumper, 2-pole, open"
+			(at 39.37 57.15 0)
+			(effects
+				(font
+					(size 1.27 1.27)
+				)
+				(hide yes)
+			)
+		)
+		(pin "2"
+		)
+		(pin "1"
+		)
+		(instances
+			(project "mcuDevBoard"
+				(path "/76df3d58-0caf-44f2-90e9-e1295852820b/5d32edae-5069-49d0-8f93-a70e744e16c2"
+					(reference "JP13")
+					(unit 1)
+				)
+				(path "/76df3d58-0caf-44f2-90e9-e1295852820b/701c2a91-874a-4ca7-8c4e-53a7a8712d0a"
+					(reference "JP14")
+					(unit 1)
+				)
